Commit message: make drive node that contains service server that pulish the service of velocity and angular of the bot

File: src/my_robot/urdf/my_robot.xacro (robot description, xacro)
@@ -40,5 +40,5 @@
         <origin xyz = "0.2 0 0" rpy = "0 0 0"/>
         <parent link = "chassis"/>
-        <child  link = "Camera"/>
+        <child  link = "camera"/>
     </joint>
     <joint name = "hokuyo_joint" type  = "fixed">
@@ -48,5 +48,5 @@
         <child  link = "hokuyo"/>
     </joint>
-    <xacro:include filename = "$(find my_robot)/urdf/my_robo.gazebo"/>
+    <xacro:include filename = "$(find my_robot)/urdf/my_robot.gazebo"/>
     <!-- LINKS -->
     <link name = "robot_footprint"></link>
@@ -138,5 +138,5 @@
         </inertial>
     </link>
-    <link name = "Camera">
+    <link name = "camera">
         <visual>
             <origin xyz = "0 0 0" rpy = "0 0 0"/>
